File: PCB/_autosave-PCB.kicad_pcb (KiCad board)
At the start: 2 copper layers, 52 parts, among them J1 12402012E212A, J2 S2B-PH-K-SLFSN, J3 Conn_01x03_Pin, Q1 SS8050, U1 ESP32-S3, U2 MCP7940MT-I_SN, U3 FSMSMTR, U4 L78M05CDT-TR, U5 MX25L6433FM2I-08Q, U6 TMC6300-LA-T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

Commit message: schematic almost ready
Parts:
- added AE1: Antenna_Shield, RF_Antenna:Texas_SWRA117D_2.4GHz_Right, F.Cu at (133.9, 21.1)
- added C28: 1.8 pF, Capacitor_SMD:C_0201_0603Metric, F.Cu at (132.0, 26.1)
- added C31: 1.2 pF, Capacitor_SMD:C_0201_0603Metric, F.Cu at (132.0, 27.9)
- added J4: Conn_01x02_Pin, Connector_JST:JST_EH_B2B-EH-A_1x02_P2.50mm_Vertical, F.Cu at (127.3, 35.5)
- added L1: 2.0 nH, Inductor_SMD:L_0603_1608Metric, F.Cu at (135.2, 26.5)
- added L3: 2.4 nH, Inductor_SMD:L_0201_0603Metric, F.Cu at (132.0, 29.6)
- added Q2: SS8050, Package_TO_SOT_SMD:SOT-23, F.Cu at (126.2, 41.1)
- added R10: 5 K, Resistor_SMD:R_0603_1608Metric, F.Cu at (130.7, 40.0)
- added R8: 10K, Resistor_SMD:R_0603_1608Metric, F.Cu at (170.0, 16.0)
- added R9: 10K, Resistor_SMD:R_0603_1608Metric, F.Cu at (170.0, 18.5)
- C20, C21, C3, C4: value 22 pF -> 15 pF
Connections:
- R7 pad 1: unconnected-(R7-Pad1) -> SDA
- R7 pad 2: unconnected-(R7-Pad2) -> +3.3V
- U1 pad 1: unconnected-(U1-LNA_IN-Pad1) -> LNA_IN
- U1 pad 6: unconnected-(U1-GPIO1-Pad6) -> LED
- U1 pad 7: unconnected-(U1-GPIO2-Pad7) -> SCL
- U1 pad 8: unconnected-(U1-GPIO3-Pad8) -> SDA
- U1 pad 9: unconnected-(U1-GPIO4-Pad9) -> MFP
