File: PCB/_autosave-PCB.kicad_sch (KiCad schematic)
At the start: 66 parts, among them J1 12402012E212A, J2 S2B-PH-K-SLFSN, J3 Conn_01x03_Pin, J4 Conn_01x02_Pin, Q1 SS8050, Q2 SS8050, U1 ESP32-S3, U2 MCP7940MT-I_SN, U3 FSMSMTR, U4 L78M05CDT-TR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

Commit message: schematic almost ready
Other:
- moved on the sheet: R7, R8
Changed lines of the file:
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@@
 	(text "I2C"
 		(exclude_from_sim no)
-		(at 91.948 64.262 0)
+		(at 560.578 344.932 0)
 		(effects
 			(font
@@
 	(wire
 		(pts
-			(xy 80.01 81.28) (xy 80.01 80.01)
+			(xy 548.64 361.95) (xy 548.64 360.68)
 		)
 		(stroke
@@
 	(wire
 		(pts
-			(xy 99.06 81.28) (xy 101.6 81.28)
+			(xy 567.69 361.95) (xy 570.23 361.95)
 		)
 		(stroke
@@
 	(wire
 		(pts
-			(xy 80.01 71.12) (xy 80.01 72.39)
+			(xy 548.64 351.79) (xy 548.64 353.06)
 		)
 		(stroke
@@
 	(wire
 		(pts
-			(xy 101.6 71.12) (xy 101.6 72.39)
+			(xy 570.23 351.79) (xy 570.23 353.06)
 		)
 		(stroke
@@
 	(wire
 		(pts
-			(xy 101.6 81.28) (xy 101.6 80.01)
+			(xy 570.23 361.95) (xy 570.23 360.68)
 		)
 		(stroke
@@
 	(wire
 		(pts
-			(xy 77.47 81.28) (xy 80.01 81.28)
+			(xy 546.1 361.95) (xy 548.64 361.95)
 		)
 		(stroke
@@
 	(global_label "SCL"
 		(shape input)
-		(at 77.47 81.28 180)
+		(at 546.1 361.95 180)
 		(fields_autoplaced yes)
 		(effects
@@
 		)
 		(property "Intersheetrefs" "${INTERSHEET_REFS}"
-			(at 70.9772 81.28 0)
+			(at 539.6072 361.95 0)
 			(effects
 				(font
@@
 	(global_label "SDA"
 		(shape input)
-		(at 99.06 81.28 180)
+		(at 567.69 361.95 180)
 		(fields_autoplaced yes)
 		(effects
@@
 		)
 		(property "Intersheetrefs" "${INTERSHEET_REFS}"
-			(at 92.5067 81.28 0)
+			(at 561.1367 361.95 0)
 			(effects
 				(font
@@
 	(symbol
 		(lib_id "power:+3.3V")
-		(at 101.6 71.12 0)
+		(at 570.23 351.79 0)
 		(unit 1)
 		(exclude_from_sim no)
@@
 		(fields_autoplaced yes)
 		(property "Reference" "#PWR063"
-			(at 101.6 74.93 0)
+			(at 570.23 355.6 0)
 			(effects
 				(font
@@
 		)
 		(property "Value" "+3.3V"
-			(at 101.6 66.04 0)
+			(at 570.23 346.71 0)
 			(effects
 				(font
@@
 		)
 		(property "Footprint" ""
-			(at 101.6 71.12 0)
+			(at 570.23 351.79 0)
 			(effects
 				(font
@@
 		)
 		(property "Datasheet" ""
-			(at 101.6 71.12 0)
+			(at 570.23 351.79 0)
 			(effects
 				(font
@@
 		)
 		(property "Description" "Power symbol creates a global label with name \"+3.3V\""
-			(at 101.6 71.12 0)
+			(at 570.23 351.79 0)
 			(effects
 				(font
@@
 	(symbol
 		(lib_id "Device:R_US")
-		(at 80.01 76.2 180)
+		(at 548.64 356.87 180)
 		(unit 1)
 		(exclude_from_sim no)
@@
 		(fields_autoplaced yes)
 		(property "Reference" "R8"
-			(at 82.55 74.9299 0)
+			(at 551.18 355.5999 0)
 			(effects
 				(font
@@
 		)
 		(property "Value" "10K"
-			(at 82.55 77.4699 0)
+			(at 551.18 358.1399 0)
 			(effects
 				(font
@@
 		)
 		(property "Footprint" "Resistor_SMD:R_0603_1608Metric"
-			(at 78.994 75.946 90)
+			(at 547.624 356.616 90)
 			(effects
 				(font
@@
 		)
 		(property "Datasheet" "~"
-			(at 80.01 76.2 0)
+			(at 548.64 356.87 0)
 			(effects
 				(font
@@
 		)
 		(property "Description" "Resistor, US symbol"
-			(at 80.01 76.2 0)
+			(at 548.64 356.87 0)
 			(effects
 				(font
@@
 	(symbol
 		(lib_id "Device:R_US")
-		(at 101.6 76.2 180)
+		(at 570.23 356.87 180)
 		(unit 1)
 		(exclude_from_sim no)
@@
 		(fields_autoplaced yes)
 		(property "Reference" "R7"
-			(at 104.14 74.9299 0)
+			(at 572.77 355.5999 0)
 			(effects
 				(font
@@
 		)
 		(property "Value" "10K"
-			(at 104.14 77.4699 0)
+			(at 572.77 358.1399 0)
 			(effects
 				(font
@@
 		)
 		(property "Footprint" "Resistor_SMD:R_0603_1608Metric"
-			(at 100.584 75.946 90)
+			(at 569.214 356.616 90)
 			(effects
 				(font
@@
 		)
 		(property "Datasheet" "~"
-			(at 101.6 76.2 0)
+			(at 570.23 356.87 0)
 			(effects
 				(font
@@
 		)
 		(property "Description" "Resistor, US symbol"
-			(at 101.6 76.2 0)
+			(at 570.23 356.87 0)
 			(effects
 				(font
@@
 	(symbol
 		(lib_id "power:+3.3V")
-		(at 80.01 71.12 0)
+		(at 548.64 351.79 0)
 		(unit 1)
 		(exclude_from_sim no)
@@
 		(fields_autoplaced yes)
 		(property "Reference" "#PWR064"
-			(at 80.01 74.93 0)
+			(at 548.64 355.6 0)
 			(effects
 				(font
@@
 		)
 		(property "Value" "+3.3V"
-			(at 80.01 66.04 0)
+			(at 548.64 346.71 0)
 			(effects
 				(font
@@
 		)
 		(property "Footprint" ""
-			(at 80.01 71.12 0)
+			(at 548.64 351.79 0)
 			(effects
 				(font
@@
 		)
 		(property "Datasheet" ""
-			(at 80.01 71.12 0)
+			(at 548.64 351.79 0)
 			(effects
 				(font
@@
 		)
 		(property "Description" "Power symbol creates a global label with name \"+3.3V\""
-			(at 80.01 71.12 0)
+			(at 548.64 351.79 0)
 			(effects
 				(font

Commit message: more pcb changes, schematic ready, now footprint
Parts:
- removed D4: D, symbol Device:D
- removed Q2: SS8050, Package_TO_SOT_SMD:SOT-23, symbol Transistor_BJT:SS8050
- removed R10: 5 K, Resistor_SMD:R_0603_1608Metric, symbol Device:R_US
- removed U4: L78M05CDT-TR, L78M05CDT_TR:VREG_L78M05CDT-TR, symbol L78M05CDT-TR:L78M05CDT-TR
- added C29: 0.1 uF, Capacitor_SMD:C_0603_1608Metric_Pad1.08x0.95mm_HandSolder, symbol Device:C
- added C30: 1 uF, Capacitor_SMD:C_0603_1608Metric_Pad1.08x0.95mm_HandSolder, symbol Device:C
- added D6: 2659, 2659:2659, symbol 2659:2659
- added J5, J6: Conn_01x09_Pin, Connector_PinHeader_2.54mm:PinHeader_1x09_P2.54mm_Vertical, symbol Connector:Conn_01x09_Pin
- added U10: LP38691SD-3.3, LP38691SD_3_3_NOPB:DFN300X300X80-7N, symbol LP38691SD-3.3:LP38691SD-3.3
- added U9: DRV2605LDGSR, DRV2605LDGSR:SOP50P490X110-10N, symbol DRV2605LDGSR:DRV2605LDGSR
- C15: value 0.1 uF -> 1 uF
- C17: value 0.33 uF -> 1 uF
- D5: footprint (none) -> LED_SMD:LED_0805_2012Metric
- R7: value 10K -> 2.2 K
- R8: value 10K -> 2.2K
Connections:
- net +3.3V: now also U10.4 (VOUT), U10.5 (SNS); no longer J4.2 (Pin_2), U1.2 (VDD3P3), U1.3 (VDD3P3__1)
- net +5V: now also C29.1, D6.4 (VDD), U10.1 (VIN_2), U10.6 (VIN)
- net GND: now also C29.2, C30.2, D6.2 (VSS), U10.2 (GND), U9.10 (VDD), U9.4 (IN/TRIG), U9.8 (GND)
- net Haptic: now also U1.23 (GPIO17), U9.5 (EN); no longer U1.18 (GPIO13)
- net RGB LED: now also U1.24 (GPIO18), D6.3 (DIN)
- net SCL: now also U9.2 (SCL)
- net SDA: now also U9.3 (SDA)
- net at J4.1 (Pin_1): now also U9.9 (OUT-)
- net 21: now reaches U1.27 (GPIO21)
- net 21: now also J6.1 (Pin_1)
- net 48: now reaches U1.36 (SPICLK_N)
- net 48: now also J5.2 (Pin_2)
- net 47: now reaches U1.37 (SPICLK_P)
- net 47: now also J5.3 (Pin_3)
- net 33: now reaches U1.38 (GPIO33)
- net 33: now also J6.2 (Pin_2)
- net 34: now reaches U1.39 (GPIO34)
- net 34: now also J6.3 (Pin_3)
- net 35: now reaches U1.40 (GPIO35)
- net 35: now also J6.4 (Pin_4)
- net 36: now reaches U1.41 (GPIO36)
- net 36: now also J6.5 (Pin_5)
- net 37: now reaches U1.42 (GPIO37)
- net 37: now also J6.6 (Pin_6)
- net 38: now reaches U1.43 (GPIO38)
- net 38: now also J6.7 (Pin_7)
- net 39: now reaches U1.44 (MTCK)
- net 39: now also J5.9 (Pin_9)
- net 40: now reaches U1.45 (MTDO)
- net 40: now also J5.8 (Pin_8)
- net 41: now reaches U1.47 (MTDI)
- net 41: now also J5.7 (Pin_7)
- net 42: now reaches U1.48 (MTMS)
- net 42: now also J5.6 (Pin_6)
- net TX: now reaches U1.49 (U0TXD)
- net TX: now also J5.4 (Pin_4)
- net RX: now reaches U1.50 (U0RXD)
- net RX: now also J5.5 (Pin_5)
- net 45: now reaches U1.51 (GPIO45)
- net 45: now also J6.8 (Pin_8)
- net 46: now reaches U1.52 (GPIO46)
- net 46: now also J6.9 (Pin_9)
- net +3.3VA: now reaches C12.1, L1.2
- net +3.3VA: now also U1.2 (VDD3P3), U1.3 (VDD3P3__1)
- new net: J4.2 (Pin_2), U9.7 (OUT+)
- new net: C30.1, U9.1 (REG)
- new net 13: J5.1 (Pin_1), U1.18 (GPIO13)
- no-connect marks 7 -> 10
Other:
- note added: "Free pins"
- note added: "RGB"
- moved on the sheet: C15, C16, C17, D1, D2, J2, J4, R7, R8
