File: PCB/PCB.kicad_pcb (KiCad board)
At the start: 2 copper layers, 52 parts, among them J1 12402012E212A, J2 S2B-PH-K-SLFSN, J3 Conn_01x03_Pin, Q1 SS8050, U1 ESP32-S3, U2 MCP7940MT-I_SN, U3 FSMSMTR, U4 L78M05CDT-TR, U5 MX25L6433FM2I-08Q, U6 TMC6300-LA-T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

Commit message: more pcb changes, schematic ready, now footprint
Parts:
- removed U4: L78M05CDT-TR, L78M05CDT_TR:VREG_L78M05CDT-TR
- added AE1: Antenna_Shield, RF_Antenna:Texas_SWRA117D_2.4GHz_Right, F.Cu at (188.6, 70.1)
- added C28: 1.8 pF, Capacitor_SMD:C_0201_0603Metric, F.Cu at (192.3, 74.2)
- added C29: 0.1 uF, Capacitor_SMD:C_0603_1608Metric_Pad1.08x0.95mm_HandSolder, F.Cu at (169.1, 61.4)
- added C30: 1 uF, Capacitor_SMD:C_0603_1608Metric_Pad1.08x0.95mm_HandSolder, F.Cu at (169.1, 63.9)
- added C31: 1.2 pF, Capacitor_SMD:C_0201_0603Metric, F.Cu at (194.7, 76.8)
- added D5: LED, LED_SMD:LED_0805_2012Metric, F.Cu at (201.5, 112.4)
- added J4: Conn_01x02_Pin, Connector_JST:JST_EH_B2B-EH-A_1x02_P2.50mm_Vertical, F.Cu at (213.8, 125.2)
- added J5: Conn_01x09_Pin, Connector_PinHeader_2.54mm:PinHeader_1x09_P2.54mm_Vertical, F.Cu at (251.8, 59.0)
- added J6: Conn_01x09_Pin, Connector_PinHeader_2.54mm:PinHeader_1x09_P2.54mm_Vertical, F.Cu at (271.0, 102.6)
- added L1: 2.0 nH, Inductor_SMD:L_0603_1608Metric, F.Cu at (191.9, 80.5)
- added L3: 2.4 nH, Inductor_SMD:L_0201_0603Metric, F.Cu at (193.8, 75.3)
- added R11: 220, Resistor_SMD:R_0603_1608Metric, F.Cu at (197.5, 109.0)
- added R8: 2.2K, Resistor_SMD:R_0603_1608Metric, F.Cu at (158.6, 101.4)
- added R9: 10K, Resistor_SMD:R_0603_1608Metric, F.Cu at (158.6, 103.9)
- added U10: LP38691SD-3.3, LP38691SD_3_3_NOPB:DFN300X300X80-7N, F.Cu at (192.0, 96.5)
- C15: value 0.1 uF -> 1 uF
- C17: value 0.33 uF -> 1 uF
- C20, C21, C3, C4: value 22 pF -> 15 pF
- R7: value 10K -> 2.2 K
- moved R2 97.8 mm to (225.5, 99.0), turned to -90 degrees
- moved C18 96.2 mm to (228.6, 101.0)
- moved R3 93.2 mm to (221.5, 98.5), turned to 180 degrees
- moved D2 92.9 mm to (199.5, 103.5), turned to 90 degrees
- moved C17 87.9 mm to (196.0, 98.5), turned to 90 degrees
- moved J1 87.8 mm to (209.7, 114.2)
- moved R4 86.3 mm to (212.5, 107.0)
- moved C21 86.2 mm to (175.3, 116.5)
- moved C23 86.2 mm to (171.1, 109.6)
- moved C24 86.2 mm to (171.1, 112.1)
- moved C26 86.2 mm to (171.0, 119.8)
- moved C27 86.2 mm to (171.1, 117.1)
- moved U2 86.2 mm to (177.8, 109.3)
- moved Y3 86.2 mm to (179.9, 120.4)
- moved C20 86.2 mm to (175.3, 114.0)
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Connections:
- C12 pad 1: Net-(C12-Pad1) -> +3.3VA
- R7 pad 1: unconnected-(R7-Pad1) -> SDA
- R7 pad 2: unconnected-(R7-Pad2) -> +3.3V
- U1 pad 1: unconnected-(U1-LNA_IN-Pad1) -> LNA_IN
- U1 pad 10: unconnected-(U1-GPIO5-Pad10) -> Buzzer
- U1 pad 11: unconnected-(U1-GPIO6-Pad11) -> UH
- U1 pad 12: unconnected-(U1-GPIO7-Pad12) -> UL
- U1 pad 13: unconnected-(U1-GPIO8-Pad13) -> VH
- U1 pad 14: unconnected-(U1-GPIO9-Pad14) -> VL
- U1 pad 15: unconnected-(U1-GPIO10-Pad15) -> WH
- U1 pad 16: unconnected-(U1-GPIO11-Pad16) -> WL
- U1 pad 17: unconnected-(U1-GPIO12-Pad17) -> DIAG
- U1 pad 18: unconnected-(U1-GPIO13-Pad18) -> 13
- U1 pad 19: unconnected-(U1-GPIO14-Pad19) -> MFP
- U1 pad 2: +3.3V -> +3.3VA
- U1 pad 23: unconnected-(U1-GPIO17-Pad23) -> Haptic
- U1 pad 24: unconnected-(U1-GPIO18-Pad24) -> RGB LED
- U1 pad 27: unconnected-(U1-GPIO21-Pad27) -> 21
- U1 pad 3: +3.3V -> +3.3VA
- U1 pad 36: unconnected-(U1-SPICLK_N-Pad36) -> 48
- U1 pad 37: unconnected-(U1-SPICLK_P-Pad37) -> 47
- U1 pad 38: unconnected-(U1-GPIO33-Pad38) -> 33
- U1 pad 39: unconnected-(U1-GPIO34-Pad39) -> 34
- U1 pad 40: unconnected-(U1-GPIO35-Pad40) -> 35
- U1 pad 41: unconnected-(U1-GPIO36-Pad41) -> 36
- U1 pad 42: unconnected-(U1-GPIO37-Pad42) -> 37
- U1 pad 43: unconnected-(U1-GPIO38-Pad43) -> 38
- U1 pad 44: unconnected-(U1-MTCK-Pad44) -> 39
- U1 pad 45: unconnected-(U1-MTDO-Pad45) -> 40
- U1 pad 47: unconnected-(U1-MTDI-Pad47) -> 41
- U1 pad 48: unconnected-(U1-MTMS-Pad48) -> 42
- U1 pad 49: unconnected-(U1-U0TXD-Pad49) -> TX
- U1 pad 50: unconnected-(U1-U0RXD-Pad50) -> RX
- U1 pad 51: unconnected-(U1-GPIO45-Pad51) -> 45
- U1 pad 52: unconnected-(U1-GPIO46-Pad52) -> 46
- U1 pad 6: unconnected-(U1-GPIO1-Pad6) -> LED
- U1 pad 7: unconnected-(U1-GPIO2-Pad7) -> SCL
- U1 pad 8: unconnected-(U1-GPIO3-Pad8) -> SDA
- U1 pad 9: unconnected-(U1-GPIO4-Pad9) -> MFP
Routing:
- net Boot: track 0.00 -> 54.0 mm, vias 0 -> 2
- net Reset: track 0.00 -> 50.9 mm
- net +3.3V: track 0.00 -> 36.4 mm
- net LED: track 0.00 -> 31.7 mm, vias 0 -> 2
- net +5VA: track 0.00 -> 27.0 mm
- net Buzzer: track 0.00 -> 22.7 mm, vias 0 -> 2
- net USB_DP: track 0.00 -> 21.5 mm
- net SPI_Q: track 0.00 -> 21.0 mm
- net USB_DN: track 0.00 -> 19.7 mm
- net SPI_CS0: track 0.00 -> 17.7 mm
- net SPI_WP: track 0.00 -> 14.7 mm
- net VS: track 0.00 -> 14.7 mm
- net USB_DP1: track 0.00 -> 8.23 mm
- net U: track 0.00 -> 7.98 mm
- net +BATT: track 0.00 -> 7.65 mm
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Other:
- board outline added: 65 x 65 mm

Commit message: first vesrion of pcb ready
Parts:
- added D6: 2659, 2659:2659, F.Cu at (208.2, 92.9)
- added U9: DRV2605LDGSR, DRV2605LDGSR:SOP50P490X110-10N, F.Cu at (198.5, 96.0)
- J5: footprint Connector_PinHeader_2.54mm:PinHeader_1x09_P2.54mm_Vertical -> Connector_PinHeader_1.27mm:PinHeader_1x09_P1.27mm_Vertical
- J6: value Conn_01x09_Pin -> Conn_01x10_Pin; footprint Connector_PinHeader_2.54mm:PinHeader_1x09_P2.54mm_Vertical -> Connector_PinHeader_1.27mm:PinHeader_1x10_P1.27mm_Vertical
- R9: value 10K -> 2.2 K
- moved J6 58.9 mm to (224.5, 66.5), turned to -125 degrees
- moved U7 54.5 mm to (181.6, 75.4), turned to -90 degrees
- moved C18 49.4 mm to (181.0, 88.0), turned to -90 degrees
- moved C29 49.2 mm to (202.0, 98.0)
- moved J3 49.2 mm to (203.0, 107.0), turned to 0 degrees
- moved U3 45.0 mm to (184.0, 94.1)
- moved C30 44.6 mm to (201.0, 95.0), turned to -90 degrees
- moved C26 43.3 mm to (211.9, 105.5), turned to -90 degrees
- moved C25 42.6 mm to (211.8, 102.3), turned to 90 degrees
- moved C22 40.7 mm to (202.0, 101.5)
- moved C24 40.4 mm to (210.3, 102.3), turned to 90 degrees
- moved R7 39.9 mm to (189.6, 84.3), turned to 180 degrees
- moved R2 39.8 mm to (187.0, 89.0), turned to 90 degrees
- moved R3 39.1 mm to (186.1, 81.8), turned to -90 degrees
- moved C19 39.1 mm to (184.5, 81.6), turned to 90 degrees
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Connections:
- D2 pad 1: +BATT -> +5VA
- D2 pad 2: +5VA -> +BATT
- J5 pad 1: 13 -> 17
- J5 pad 2: 48 -> 18
- J5 pad 3: 47 -> 21
- J5 pad 4: TX -> 48
- J5 pad 5: RX -> 47
- J5 pad 6: 42 -> 33
- J5 pad 7: 41 -> 34
- J5 pad 8: 40 -> 35
- J5 pad 9: 39 -> 36
- J6 pad 1: 21 -> 37
- J6 pad 2: 33 -> 38
- J6 pad 3: 34 -> 39
- J6 pad 4: 35 -> 40
- J6 pad 5: 36 -> 41
- J6 pad 6: 37 -> 42
- J6 pad 7: 38 -> TX
- J6 pad 8: 45 -> RX
- J6 pad 9: 46 -> 45
- U1 pad 10: Buzzer -> Haptic
- U1 pad 11: UH -> VL
- U1 pad 12: UL -> WL
- U1 pad 13: VH -> UL
- U1 pad 14: VL -> WH
- U1 pad 15: WH -> VH
- U1 pad 16: WL -> UH
- U1 pad 18: 13 -> Buzzer
- U1 pad 19: MFP -> RGB LED
- U1 pad 23: Haptic -> 17
- U1 pad 24: RGB LED -> 18
- U1 pad 58: (no net) -> GND
- U1 pad 59: (no net) -> GND
- U1 pad 60: (no net) -> GND
- U1 pad 61: (no net) -> GND
- U1 pad 62: (no net) -> GND
- U1 pad 63: (no net) -> GND
- U1 pad 64: (no net) -> GND
- U1 pad 65: (no net) -> GND
- U1 pad 66: (no net) -> GND
- U1 pad 67: (no net) -> GND
- U1 pad 68: (no net) -> GND
- U1 pad 69: (no net) -> GND
Routing:
- net +3.3V: track 36.4 -> 127.5 mm, vias 0 -> 7
- net GND: track 0.00 -> 63.3 mm, vias 0 -> 168
- net 17: track 0.00 -> 36.2 mm
- net 18: track 0.00 -> 35.4 mm
- net Reset: track 50.9 -> 16.2 mm
- net 21: track 0.00 -> 33.5 mm, vias 0 -> 2
- net Boot: track 54.0 -> 22.5 mm, vias 2 -> 0
- net VS: track 14.7 -> 45.9 mm, vias 0 -> 4
- net 41: track 0.00 -> 30.5 mm, vias 0 -> 4
- net 40: track 0.00 -> 28.9 mm, vias 0 -> 2
- net 48: track 0.00 -> 28.8 mm, vias 0 -> 2
- net 47: track 0.00 -> 28.7 mm, vias 0 -> 2
- net 33: track 0.00 -> 28.6 mm, vias 0 -> 2
- net 34: track 0.00 -> 28.6 mm, vias 0 -> 2
- net 35: track 0.00 -> 28.5 mm, vias 0 -> 2
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- added copper zone on B.Cu, net GND
- added copper zone on F.Cu, net GND
Other:
- board size 65 x 65 mm -> 54.1 x 54.1 mm

Commit message: last changes for the pcb
Parts:
- removed AE1: Antenna_Shield, RF_Antenna:Texas_SWRA117D_2.4GHz_Right
- removed C20, C21, C3, C4: 15 pF, Capacitor_SMD:C_0603_1608Metric
- removed U3, U7: FSMSMTR, FSMSMTR:SWITCH_FSMSMTR_TYC
- removed U5: MX25L6433FM2I-08Q, mx flash:SOP8_200MIL_MAC-M
- removed Y1, Y3: ABS07-32.768KHZ-T, ABS07_32_768KHZ_T(1):XTAL_ABS07-32.768KHZ-T
- added CR1: KSS231G LFS, KSS231G:SW_KSS2, F.Cu at (248.0, 98.0)
- added CR2: KSS231G LFS, KSS231G:SW_KSS2, F.Cu at (241.1, 58.0)
- added CR3: KSS231G LFS, KSS231G:SW_KSS2, F.Cu at (241.1, 64.0)
- added E1: AMCA31-2R450G-S1F-T3, AMCA31_2R450G_S1F_T3:XDCR_AMCA31-2R450G-S1F-T3, F.Cu at (240.3, 111.0)
- added R10: 2.2 K, Resistor_SMD:R_0201_0603Metric_Pad0.64x0.40mm_HandSolder, F.Cu at (227.8, 60.8)
- added U11: BME688, BME688:IC_BME688, F.Cu at (238.8, 82.8)
- added U12: RV-3028-C7_32.768KHZ_1PPM-TA-QC, Package_SON:MicroCrystal_C7_SON-8_1.5x3.2mm_P0.9mm, F.Cu at (241.3, 73.5)
- added U13: LTR-329ALS-01, LTR_329ALS_01:IC_LTR-329ALS-01, F.Cu at (252.3, 75.4)
- added U14: BQ27427YZFR, BQ27427YZFR:IC_BQ27427YZFR, F.Cu at (242.5, 90.5)
- added U15: MCP73832T-2ACI/MC, MCP73832T:DFN8_2x3MC_MCH-L, F.Cu at (260.7, 90.2)
- added U16: LSM6DSO32TR, LSM6DSO32TR:XDCR_LSM6DSO32TR, F.Cu at (250.8, 89.2)
- C1, C10, C11, C12, C13, C14, C15, C17, C18, C19, C22, C23, C24, C25, C27, C29, C30, C7, C8, C9: footprint Capacitor_SMD:C_0603_1608Metric_Pad1.08x0.95mm_HandSolder -> Capacitor_SMD:C_0201_0603Metric_Pad0.64x0.40mm_HandSolder
- C16, C2, C26: footprint Capacitor_Tantalum_SMD:CP_EIA-1608-08_AVX-J -> Capacitor_Tantalum_SMD:CP_EIA-1608-08_AVX-J_HandSolder
- C5, C6: footprint Capacitor_SMD:C_0603_1608Metric -> Capacitor_SMD:C_0201_0603Metric_Pad0.64x0.40mm_HandSolder
- J2: footprint jst:CONN_S2B-PH-K-S_JST -> Connector_JST:JST_ZH_B2B-ZR_1x02_P1.50mm_Vertical
- J3: footprint Connector_JST:JST_EH_B3B-EH-A_1x03_P2.50mm_Vertical -> Connector_JST:JST_ZH_B3B-ZR_1x03_P1.50mm_Vertical
- J4: footprint Connector_JST:JST_EH_B2B-EH-A_1x02_P2.50mm_Vertical -> Connector_JST:JST_ZH_B2B-ZR_1x02_P1.50mm_Vertical
- L1: footprint Inductor_SMD:L_0603_1608Metric -> Inductor_SMD:L_0201_0603Metric_Pad0.64x0.40mm_HandSolder
- R1, R11, R2, R3, R4, R5, R6: footprint Resistor_SMD:R_0603_1608Metric -> Resistor_SMD:R_0201_0603Metric_Pad0.64x0.40mm_HandSolder
- R7, R9: value 2.2 K -> 10 K; footprint Resistor_SMD:R_0603_1608Metric -> Resistor_SMD:R_0201_0603Metric_Pad0.64x0.40mm_HandSolder
- R8: value 2.2K -> 10 K; footprint Resistor_SMD:R_0603_1608Metric -> Resistor_SMD:R_0201_0603Metric_Pad0.64x0.40mm_HandSolder
- U2: value MCP7940MT-I_SN -> MX25R6435FZAIH0; footprint MCP7940MT_I_SN:SOIC127P600X175-8N -> MX25R6435FZAIH0:SON80P400X400X60-9N
- moved U2 18.1 mm to (208.1, 81.6), turned to 0 degrees
Connections:
- U1 pad 58: GND -> (no net)
- U1 pad 59: GND -> (no net)
- U1 pad 60: GND -> (no net)
- U1 pad 61: GND -> (no net)
- U1 pad 62: GND -> (no net)
- U1 pad 63: GND -> (no net)
- U1 pad 64: GND -> (no net)
- U1 pad 65: GND -> (no net)
- U1 pad 66: GND -> (no net)
- U1 pad 67: GND -> (no net)
- U1 pad 68: GND -> (no net)
- U1 pad 69: GND -> (no net)
- U2 pad 1: X1 -> unconnected-(U2-CS#-Pad1)
- U2 pad 2: X2 -> unconnected-(U2-SO/SIO1-Pad2)
- U2 pad 3: (no net) -> unconnected-(U2-WP#/SIO2-Pad3)
- U2 pad 4: GND -> unconnected-(U2-GND-Pad4)
- U2 pad 5: SDA -> unconnected-(U2-SI/SIO0-Pad5)
- U2 pad 6: SCL -> unconnected-(U2-SCLK-Pad6)
- U2 pad 7: MFP -> unconnected-(U2-RESET#/SIO3-Pad7)
- U2 pad 8: +3.3V -> unconnected-(U2-VCC-Pad8)
Routing:
- net (no net): track 0.00 -> 10.5 mm
- net X1: track 5.72 -> 0.00 mm
- net X2: track 4.78 -> 0.00 mm
Other:
- board size 54.1 x 54.1 mm -> 104 x 54.1 mm
