File: PCB/PCB.kicad_sch (KiCad schematic)
At the start: 66 parts, among them J1 12402012E212A, J2 S2B-PH-K-SLFSN, J3 Conn_01x03_Pin, J4 Conn_01x02_Pin, Q1 SS8050, Q2 SS8050, U1 ESP32-S3, U2 MCP7940MT-I_SN, U3 FSMSMTR, U4 L78M05CDT-TR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

Commit message: more pcb changes, schematic ready, now footprint
Parts:
- removed D4: D, symbol Device:D
- removed Q2: SS8050, Package_TO_SOT_SMD:SOT-23, symbol Transistor_BJT:SS8050
- removed R10: 5 K, Resistor_SMD:R_0603_1608Metric, symbol Device:R_US
- removed U4: L78M05CDT-TR, L78M05CDT_TR:VREG_L78M05CDT-TR, symbol L78M05CDT-TR:L78M05CDT-TR
- added C29: 0.1 uF, Capacitor_SMD:C_0603_1608Metric_Pad1.08x0.95mm_HandSolder, symbol Device:C
- added C30: 1 uF, Capacitor_SMD:C_0603_1608Metric_Pad1.08x0.95mm_HandSolder, symbol Device:C
- added D6: 2659, 2659:2659, symbol 2659:2659
- added J5, J6: Conn_01x09_Pin, Connector_PinHeader_2.54mm:PinHeader_1x09_P2.54mm_Vertical, symbol Connector:Conn_01x09_Pin
- added U10: LP38691SD-3.3, LP38691SD_3_3_NOPB:DFN300X300X80-7N, symbol LP38691SD-3.3:LP38691SD-3.3
- added U9: DRV2605LDGSR, DRV2605LDGSR:SOP50P490X110-10N, symbol DRV2605LDGSR:DRV2605LDGSR
- C15: value 0.1 uF -> 1 uF
- C17: value 0.33 uF -> 1 uF
- D5: footprint (none) -> LED_SMD:LED_0805_2012Metric
- R7: value 10K -> 2.2 K
- R8: value 10K -> 2.2K
Connections:
- net +3.3V: now also U10.4 (VOUT), U10.5 (SNS); no longer J4.2 (Pin_2), U1.2 (VDD3P3), U1.3 (VDD3P3__1)
- net +5V: now also C29.1, D6.4 (VDD), U10.1 (VIN_2), U10.6 (VIN)
- net GND: now also C29.2, C30.2, D6.2 (VSS), U10.2 (GND), U9.10 (VDD), U9.4 (IN/TRIG), U9.8 (GND)
- net Haptic: now also U1.23 (GPIO17), U9.5 (EN); no longer U1.18 (GPIO13)
- net RGB LED: now also U1.24 (GPIO18), D6.3 (DIN)
- net SCL: now also U9.2 (SCL)
- net SDA: now also U9.3 (SDA)
- net at J4.1 (Pin_1): now also U9.9 (OUT-)
- net 21: now reaches U1.27 (GPIO21)
- net 21: now also J6.1 (Pin_1)
- net 48: now reaches U1.36 (SPICLK_N)
- net 48: now also J5.2 (Pin_2)
- net 47: now reaches U1.37 (SPICLK_P)
- net 47: now also J5.3 (Pin_3)
- net 33: now reaches U1.38 (GPIO33)
- net 33: now also J6.2 (Pin_2)
- net 34: now reaches U1.39 (GPIO34)
- net 34: now also J6.3 (Pin_3)
- net 35: now reaches U1.40 (GPIO35)
- net 35: now also J6.4 (Pin_4)
- net 36: now reaches U1.41 (GPIO36)
- net 36: now also J6.5 (Pin_5)
- net 37: now reaches U1.42 (GPIO37)
- net 37: now also J6.6 (Pin_6)
- net 38: now reaches U1.43 (GPIO38)
- net 38: now also J6.7 (Pin_7)
- net 39: now reaches U1.44 (MTCK)
- net 39: now also J5.9 (Pin_9)
- net 40: now reaches U1.45 (MTDO)
- net 40: now also J5.8 (Pin_8)
- net 41: now reaches U1.47 (MTDI)
- net 41: now also J5.7 (Pin_7)
- net 42: now reaches U1.48 (MTMS)
- net 42: now also J5.6 (Pin_6)
- net TX: now reaches U1.49 (U0TXD)
- net TX: now also J5.4 (Pin_4)
- net RX: now reaches U1.50 (U0RXD)
- net RX: now also J5.5 (Pin_5)
- net 45: now reaches U1.51 (GPIO45)
- net 45: now also J6.8 (Pin_8)
- net 46: now reaches U1.52 (GPIO46)
- net 46: now also J6.9 (Pin_9)
- net +3.3VA: now reaches C12.1, L1.2
- net +3.3VA: now also U1.2 (VDD3P3), U1.3 (VDD3P3__1)
- new net: J4.2 (Pin_2), U9.7 (OUT+)
- new net: C30.1, U9.1 (REG)
- new net 13: J5.1 (Pin_1), U1.18 (GPIO13)
- no-connect marks 7 -> 10
Other:
- note added: "Free pins"
- note added: "RGB"
- moved on the sheet: C15, C16, C17, D1, D2, J2, J4, R7, R8

Commit message: first vesrion of pcb ready
Parts:
- removed J6: Conn_01x09_Pin, Connector_PinHeader_2.54mm:PinHeader_1x09_P2.54mm_Vertical, symbol Connector:Conn_01x09_Pin
- added J6: Conn_01x10_Pin, Connector_PinHeader_1.27mm:PinHeader_1x10_P1.27mm_Vertical, symbol Connector:Conn_01x10_Pin
- J5: footprint Connector_PinHeader_2.54mm:PinHeader_1x09_P2.54mm_Vertical -> Connector_PinHeader_1.27mm:PinHeader_1x09_P1.27mm_Vertical
- R9: value 10K -> 2.2 K
Connections:
- net +5V: now also U9.10 (VDD)
- net +5VA: now also D2.1; no longer D2.2
- net +BATT: now also D2.2; no longer D2.1
- net 21: now also J5.3 (Pin_3)
- net 33: now also J5.6 (Pin_6)
- net 34: now also J5.7 (Pin_7)
- net 35: now also J5.8 (Pin_8)
- net 36: now also J5.9 (Pin_9)
- net 37: now also J6.1 (Pin_1)
- net 38: now also J6.2 (Pin_2)
- net 39: now also J6.3 (Pin_3); no longer J5.9 (Pin_9)
- net 40: now also J6.4 (Pin_4); no longer J5.8 (Pin_8)
- net 41: now also J6.5 (Pin_5); no longer J5.7 (Pin_7)
- net 42: now also J6.6 (Pin_6); no longer J5.6 (Pin_6)
- net 45: now also J6.9 (Pin_9)
- net 46: now also J6.10 (Pin_10)
- net 47: now also J5.5 (Pin_5); no longer J5.3 (Pin_3)
- net 48: now also J5.4 (Pin_4); no longer J5.2 (Pin_2)
- net Buzzer: now also U1.18 (GPIO13); no longer U1.10 (GPIO5)
- net GND: no longer U9.10 (VDD)
- net Haptic: now also U1.10 (GPIO5); no longer U1.23 (GPIO17)
- net MFP: no longer U1.19 (GPIO14)
- net RGB LED: now also U1.19 (GPIO14); no longer U1.24 (GPIO18)
- net RX: now also J6.8 (Pin_8); no longer J5.5 (Pin_5)
- net TX: now also J6.7 (Pin_7); no longer J5.4 (Pin_4)
- net UH: now also U1.16 (GPIO11); no longer U1.11 (GPIO6)
- net UL: now also U1.13 (GPIO8); no longer U1.12 (GPIO7)
- net VH: now also U1.15 (GPIO10); no longer U1.13 (GPIO8)
- net VL: now also U1.11 (GPIO6); no longer U1.14 (GPIO9)
- net WH: now also U1.14 (GPIO9); no longer U1.15 (GPIO10)
- net WL: now also U1.12 (GPIO7); no longer U1.16 (GPIO11)
- net at J4.1 (Pin_1): now also U9.7 (OUT+); no longer U9.9 (OUT-)
- net at J4.2 (Pin_2): now also U9.9 (OUT-); no longer U9.7 (OUT+)
- net 13 renamed 17
- net 17: now also U1.23 (GPIO17); no longer U1.18 (GPIO13)
- new net 18: J5.2 (Pin_2), U1.24 (GPIO18)
Other:
- note removed: "resistor?"
- moved on the sheet: J4

Commit message: last changes for the pcb
Parts:
- removed AE1: Antenna_Shield, RF_Antenna:Texas_SWRA117D_2.4GHz_Right, symbol Device:Antenna_Shield
- removed C20, C21, C3, C4: 15 pF, Capacitor_SMD:C_0603_1608Metric, symbol Device:C
- removed U2: MCP7940MT-I_SN, MCP7940MT_I_SN:SOIC127P600X175-8N, symbol MCP7940MT-I_SN:MCP7940MT-I_SN
- removed U3, U7: FSMSMTR, FSMSMTR:SWITCH_FSMSMTR_TYC, symbol FSMSMTR:FSMSMTR
- removed U5: MX25L6433FM2I-08Q, mx flash:SOP8_200MIL_MAC-M, symbol flash memory:MX25L6433FM2I-08Q
- removed Y1, Y3: ABS07-32.768KHZ-T, ABS07_32_768KHZ_T(1):XTAL_ABS07-32.768KHZ-T, symbol ABS07-32.768KHZ-T:ABS07-32.768KHZ-T
- added CR1, CR2, CR3: KSS231G LFS, KSS231G:SW_KSS2, symbol KSS231G:KSS231G_LFS
- added E1: AMCA31-2R450G-S1F-T3, AMCA31_2R450G_S1F_T3:XDCR_AMCA31-2R450G-S1F-T3, symbol AMCA31-2R450G-S1F-T3:AMCA31-2R450G-S1F-T3
- added R10: 2.2 K, Resistor_SMD:R_0201_0603Metric_Pad0.64x0.40mm_HandSolder, symbol Device:R_US
- added U11: BME688, BME688:IC_BME688, symbol BME688:BME688
- added U12: RV-3028-C7_32.768KHZ_1PPM-TA-QC, Package_SON:MicroCrystal_C7_SON-8_1.5x3.2mm_P0.9mm, symbol RV-3028-C7_32.768KHZ_1PPM-TA-QC:RV-3028-C7_32.768KHZ_1PPM-TA-QC
- added U13: LTR-329ALS-01, LTR_329ALS_01:IC_LTR-329ALS-01, symbol LTR-329ALS-01:LTR-329ALS-01
- added U14: BQ27427YZFR, BQ27427YZFR:IC_BQ27427YZFR, symbol BQ27427YZFR:BQ27427YZFR
- added U15: MCP73832T-2ACI/MC, MCP73832T:DFN8_2x3MC_MCH-L, symbol MCP73832T_2ACI:MCP73832T-2ACI_MC
- added U16: LSM6DSO32TR, LSM6DSO32TR:XDCR_LSM6DSO32TR, symbol LSM6DSO32TR:LSM6DSO32TR
- added U2: MX25R6435FZAIH0, MX25R6435FZAIH0:SON80P400X400X60-9N, symbol MX25R6435FZAIH0:MX25R6435FZAIH0
- C1, C10, C11, C12, C13, C14, C15, C17, C18, C19, C22, C23, C24, C25, C27, C29, C30, C7, C8, C9: footprint Capacitor_SMD:C_0603_1608Metric_Pad1.08x0.95mm_HandSolder -> Capacitor_SMD:C_0201_0603Metric_Pad0.64x0.40mm_HandSolder
- C16, C2, C26: footprint Capacitor_Tantalum_SMD:CP_EIA-1608-08_AVX-J -> Capacitor_Tantalum_SMD:CP_EIA-1608-08_AVX-J_HandSolder
- C5, C6: footprint Capacitor_SMD:C_0603_1608Metric -> Capacitor_SMD:C_0201_0603Metric_Pad0.64x0.40mm_HandSolder
- D6: MPN (none) -> 1528-2659-ND
- J2: footprint jst:CONN_S2B-PH-K-S_JST -> Connector_JST:JST_ZH_B2B-ZR_1x02_P1.50mm_Vertical
- J3: footprint Connector_JST:JST_EH_B3B-EH-A_1x03_P2.50mm_Vertical -> Connector_JST:JST_ZH_B3B-ZR_1x03_P1.50mm_Vertical
- J4: footprint Connector_JST:JST_EH_B2B-EH-A_1x02_P2.50mm_Vertical -> Connector_JST:JST_ZH_B2B-ZR_1x02_P1.50mm_Vertical
- L1: footprint Inductor_SMD:L_0603_1608Metric -> Inductor_SMD:L_0201_0603Metric_Pad0.64x0.40mm_HandSolder
- R1, R11, R2, R3, R4, R5, R6: footprint Resistor_SMD:R_0603_1608Metric -> Resistor_SMD:R_0201_0603Metric_Pad0.64x0.40mm_HandSolder
- R7, R9: value 2.2 K -> 10 K; footprint Resistor_SMD:R_0603_1608Metric -> Resistor_SMD:R_0201_0603Metric_Pad0.64x0.40mm_HandSolder
- R8: value 2.2K -> 10 K; footprint Resistor_SMD:R_0603_1608Metric -> Resistor_SMD:R_0201_0603Metric_Pad0.64x0.40mm_HandSolder
- U6: MPN (none) -> 175-TMC6300-LA-TCT-ND
Connections:
- net GND: now also CR2.1, CR3.1, R10.1, U12.5 (VSS)
- net MFP: now also U12.2 (~{INT})
- net SCL: now also U12.3 (SCL)
- net SDA: now also U12.4 (SDA)
- net at C28.2, L3.1: now also E1.1
- new net EVI: R10.2, U12.8 (EVI)
Other:
- note added: "Battery control"
- note added: "IMU"
- note added: "Light sensor"
- note added: "Temp and humidity"
- note added: "battery charger"
- note added: "battery gauge"
- note removed: "32KHz"
- moved on the sheet: C18, C19, J5, J6, R2
