File: PCB/TOP-PCB/TOP-PCB.kicad_sch (KiCad schematic)
At the start: 85 parts, among them J1 12402012E212A, J2 S2B-PH-K-SLFSN, J3 Conn_01x03_Pin, J5 Conn_01x12_Pin, Q1 QM6006D, Q2 NPN, SW2 PTS810_SJM_250_SMTR_LFS, SW3 PTS810_SJM_250_SMTR_LFS, U1 ESP32-S3, U10 LP38691SD-3.3, U11 BME688, U12 RV-3028-C7_32.768KHZ_1PPM-TA-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, U13 LTR-329ALS-01, U14 BQ27427YZFR, U15 MCP73832T-2ACI/MC, U16 LSM6DSO32TR, U2 MX25R6435FZAIH0, U3 DRV2605LYZFR, U4 MLX90393SLW-ABA-011-RE, U6 TMC6300-LA-T, U8 USBLC6-2SC6, Y1 ABM12W-40.0000MHZ-8-B1U-T3

Commit message: re organization of top and bottom pcb
Parts:
- removed C1, C11, C14, C15, C17: 1 uF, Capacitor_SMD:C_0201_0603Metric_Pad0.64x0.40mm_HandSolder, symbol Device:C
- removed C10, C12, C18, C19, C20, C22, C23, C24, C25, C27, C34, C4, C7, C8, C9: 0.1 uF, Capacitor_SMD:C_0201_0603Metric_Pad0.64x0.40mm_HandSolder, symbol Device:C
- removed C13: 10 nF, Capacitor_SMD:C_0201_0603Metric_Pad0.64x0.40mm_HandSolder, symbol Device:C
- removed C16, C2: 10 uF, Capacitor_Tantalum_SMD:CP_EIA-1608-08_AVX-J_HandSolder, symbol Device:C_Polarized
- removed C21, C29: 1 uF, Capacitor_SMD:C_0201_0603Metric, symbol Device:C
- removed C26: 22 uF, Capacitor_Tantalum_SMD:CP_EIA-1608-08_AVX-J_HandSolder, symbol Device:C_Polarized
- removed C28: 1.8 pF, Capacitor_SMD:C_0201_0603Metric, symbol Device:C
- removed C30, C32: 4.7 uF, Capacitor_SMD:C_0201_0603Metric, symbol Device:C
- removed C31: 1.5 pF, Capacitor_SMD:C_0201_0603Metric, symbol Device:C
- removed C33: 2.2 uF, Capacitor_SMD:C_0201_0603Metric, symbol Device:C
- removed C35: 22 uF, Capacitor_SMD:C_0201_0603Metric_Pad0.64x0.40mm_HandSolder, symbol Device:C
- removed C5, C6: 6 pF, Capacitor_SMD:C_0201_0603Metric_Pad0.64x0.40mm_HandSolder, symbol Device:C
- removed D1: SD03_SOD323, Diode_SMD:D_SOD-323, symbol Diode:SD05_SOD323
- removed D2: BAT54C, Package_TO_SOT_SMD:SOT-23, symbol Diode:BAT54C
- removed D3: D, symbol Device:D
- removed D4, D5: LED, LED_SMD:LED_0805_2012Metric, symbol Device:LED
- removed E1: AMCA31-2R450G-S1F-T3, AMCA31_2R450G_S1F_T3:XDCR_AMCA31-2R450G-S1F-T3, symbol AMCA31-2R450G-S1F-T3:AMCA31-2R450G-S1F-T3
- removed J1: 12402012E212A, 12402012E212A:AMPHENOL_12402012E212A, symbol 12402012E212A:12402012E212A
- removed J2: S2B-PH-K-SLFSN, Connector_JST:JST_ZH_B2B-ZR_1x02_P1.50mm_Vertical, symbol jst:S2B-PH-K-SLFSN
- removed J3: Conn_01x03_Pin, Connector_JST:JST_ZH_B3B-ZR_1x03_P1.50mm_Vertical, symbol Connector:Conn_01x03_Pin
- removed J5: Conn_01x12_Pin, GC9A01:GC9A01Round1.28, symbol Connector:Conn_01x12_Pin
- removed L1: 2.0 nH, Inductor_SMD:L_0201_0603Metric_Pad0.64x0.40mm_HandSolder, symbol Device:L
- removed L3: 3.9 nH, Inductor_SMD:L_0201_0603Metric, symbol Device:L
- removed LS2: CMT-0525-75-SMT-TR, CMT_0525_75_SMT_TR:XDCR_CMT-0525-75-SMT-TR, symbol CMT-0525-75-SMT-TR:CMT-0525-75-SMT-TR
- removed Q2: NPN, Package_TO_SOT_SMD:SOT-723, symbol Simulation_SPICE:NPN
- removed R10, R15, R16, R7, R8, R9: 10 K, Resistor_SMD:R_0201_0603Metric_Pad0.64x0.40mm_HandSolder, symbol Device:R_US
- removed R11: 220, Resistor_SMD:R_0201_0603Metric_Pad0.64x0.40mm_HandSolder, symbol Device:R_US
- removed R12: 470, Resistor_SMD:R_0201_0603Metric_Pad0.64x0.40mm_HandSolder, symbol Device:R_US
- removed R13: 2k, Resistor_SMD:R_0201_0603Metric_Pad0.64x0.40mm_HandSolder, symbol Device:R_US
- removed R14: 10k, Resistor_SMD:R_0201_0603Metric_Pad0.64x0.40mm_HandSolder, symbol Device:R_US
- removed R17: 1 M, Resistor_SMD:R_0201_0603Metric_Pad0.64x0.40mm_HandSolder, symbol Device:R_US
- removed R18: 22R, Resistor_SMD:R_0201_0603Metric_Pad0.64x0.40mm_HandSolder, symbol Device:R_US
- removed R4, R5, R6: 5 K, Resistor_SMD:R_0201_0603Metric_Pad0.64x0.40mm_HandSolder, symbol Device:R_US
- removed S1: B3F-4055, B3F_4055:SW_B3F-4055, symbol B3F-4055:B3F-4055
- removed SW2, SW3: PTS810_SJM_250_SMTR_LFS, PTS810SJM250SMTR_LFS:SW_PTS810_SJM_250_SMTR_LFS, symbol PTS810_SJM_250_SMTR_LFS:PTS810_SJM_250_SMTR_LFS
- removed U1: ESP32-S3, ESP32_S3:IC_ESP32-S3, symbol ESP32-S3:ESP32-S3
- removed U10: LP38691SD-3.3, LP38691SD_3_3_NOPB:DFN300X300X80-7N, symbol LP38691SD-3.3:LP38691SD-3.3
- removed U11: BME688, BME688:IC_BME688, symbol BME688:BME688
- removed U12: RV-3028-C7_32.768KHZ_1PPM-TA-QC, Package_SON:MicroCrystal_C7_SON-8_1.5x3.2mm_P0.9mm, symbol RV-3028-C7_32.768KHZ_1PPM-TA-QC:RV-3028-C7_32.768KHZ_1PPM-TA-QC
- removed U13: LTR-329ALS-01, LTR_329ALS_01:IC_LTR-329ALS-01, symbol LTR-329ALS-01:LTR-329ALS-01
- removed U14: BQ27427YZFR, BQ27427YZFR:IC_BQ27427YZFR, symbol BQ27427YZFR:BQ27427YZFR
- removed U15: MCP73832T-2ACI/MC, MCP73832T:DFN8_2x3MC_MCH-L, symbol MCP73832T_2ACI:MCP73832T-2ACI_MC
- removed U16: LSM6DSO32TR, LSM6DSO32TR:XDCR_LSM6DSO32TR, symbol LSM6DSO32TR:LSM6DSO32TR
- removed U2: MX25R6435FZAIH0, MX25R6435FZAIH0:SON80P400X400X60-9N, symbol MX25R6435FZAIH0:MX25R6435FZAIH0
- removed U3: DRV2605LYZFR, DRV2605LYZFR:YZF0009ADAD, symbol DRV2605LYZFR:DRV2605LYZFR
- removed U4: MLX90393SLW-ABA-011-RE, MLX90393SLW_ABA_011_RE:QFN50P300X300X100-17N, symbol MLX90393SLW-ABA-011-RE:MLX90393SLW-ABA-011-RE
- removed U6: TMC6300-LA-T, tcm6300:21-100586_K2033&plus_1C_ADI-M, symbol tcm6300:TMC6300-LA-T
- removed U8: USBLC6-2SC6, Package_TO_SOT_SMD:SOT-23-6, symbol Power_Protection:USBLC6-2SC6
- removed Y1: ABM12W-40.0000MHZ-8-B1U-T3, ABM12W_40_0000MHZ_8_B1U_T3:XTAL_ABM12W-40.0000MHZ-8-B1U-T3, symbol ABM12W-40.0000MHZ-8-B1U-T3:ABM12W-40.0000MHZ-8-B1U-T3
- added C2: 22 uF, Capacitor_SMD:C_0201_0603Metric_Pad0.64x0.40mm_HandSolder, symbol Device:C
- added J1, J2: Conn_01x04_Pin, Connector_PinHeader_1.27mm:PinHeader_1x04_P1.27mm_Vertical, symbol Connector:Conn_01x04_Pin
- added J3: Conn_01x12_Pin, LCD_GC9A01:GC9A01Round1.28, symbol Connector:Conn_01x12_Pin
- C3: value 0.1 uF -> 22 uF
- R1: value 0 -> 22R
- R2, R3: value 5 K -> 22R
Connections:
- net Boot is gone; now on an unnamed net: R2.2
- net Reset is gone; now on net GND: R3.2
- net XTAL_P is gone; now on net LEDA: R1.2
- net +3.3V: now also R1.1, C2.1, J1.1 (Pin_1), J3.4 (Pin_4); no longer R2.1, R3.1
- net DC: now also J1.4 (Pin_4), J3.7 (Pin_7)
- net GND: now also C2.2, J1.2 (Pin_2), J3.1 (Pin_1), J3.12 (Pin_12), J3.5 (Pin_5), J3.6 (Pin_6)
- net LEDA: now also J3.3 (Pin_3)
- net LEDK: now also J3.2 (Pin_2)
- net MOSI: now also J2.3 (Pin_3), J3.10 (Pin_10)
- net SCK: now also J2.2 (Pin_2), J3.9 (Pin_9)
- net nCS: now also J2.1 (Pin_1), J3.8 (Pin_8)
- net nRESET: now also J2.4 (Pin_4), J3.11 (Pin_11)
- net at Q1.1 (G): now also R3.1
- new net BACKLIGH_EN: J1.3 (Pin_3), R2.1
- no-connect marks 15 -> 0
Other:
- note added: "PCB 0.6 mm thick"
- note removed: "Antenna"
- note removed: "Battery control"
- note removed: "Buzzer"
- note removed: "Crystals"
- note removed: "Encoder"
- note removed: "Flash and PSRAM(optional)"
- note removed: "Haptic engine"
- note removed: "I2C"
- note removed: "IMU"
- note removed: "Light sensor"
- note removed: "Microcontroller"
- note removed: "Motor"
- note removed: "Power supply"
- note removed: "Power up"
- note removed: "RGB"
- note removed: "RTC module"
- note removed: "Screen"
- note removed: "Temp and humidity"
- note removed: "USB"
- note removed: "User interaction"
- note removed: "battery charger"
- note removed: "battery gauge"
- note removed: "button must be connected to pin capable of pull up"
- note removed: "could add current sensing and on/off control if needed"
