File: PCB/BOTTOM-PCB/BOTTOM-PCB.kicad_sch (KiCad schematic)
At the start: 8 parts, among them J1 Conn_01x10_Pin, J2 Conn_01x03_Pin, J3 Conn_01x02_Pin, U1 MLX90393SLW-ABA-011-RE

Commit message: re organization of top and bottom pcb
Parts:
- removed C2: 0.1uF, Capacitor_SMD:C_0603_1608Metric_Pad1.08x0.95mm_HandSolder, symbol Device:C
- removed J1: Conn_01x10_Pin, 8_188275_0:TE_8-188275-0, symbol Connector:Conn_01x10_Pin
- removed J2: Conn_01x03_Pin, Connector_JST:JST_EH_B3B-EH-A_1x03_P2.50mm_Vertical, symbol Connector:Conn_01x03_Pin
- removed J3: Conn_01x02_Pin, Connector_JST:JST_EH_B2B-EH-A_1x02_P2.50mm_Vertical, symbol Connector:Conn_01x02_Pin
- removed R1: 5K, Resistor_SMD:R_0603_1608Metric_Pad0.98x0.95mm_HandSolder, symbol Device:R_Small_US
- removed U1: MLX90393SLW-ABA-011-RE, MLX90393SLW_ABA_011_RE:QFN50P300X300X100-17N, symbol MLX90393SLW-ABA-011-RE:MLX90393SLW-ABA-011-RE
- added C10, C12, C18, C19, C20, C22, C23, C24, C25, C27, C3, C37, C4, C7, C8, C9: 0.1 uF, Capacitor_SMD:C_0201_0603Metric_Pad0.64x0.40mm_HandSolder, symbol Device:C
- added C11, C14, C15, C17: 1 uF, Capacitor_SMD:C_0201_0603Metric_Pad0.64x0.40mm_HandSolder, symbol Device:C
- added C13: 10 nF, Capacitor_SMD:C_0201_0603Metric_Pad0.64x0.40mm_HandSolder, symbol Device:C
- added C16, C2: 10 uF, Capacitor_Tantalum_SMD:CP_EIA-1608-08_AVX-J_HandSolder, symbol Device:C_Polarized
- added C21, C29: 1 uF, Capacitor_SMD:C_0201_0603Metric, symbol Device:C
- added C26: 22 uF, Capacitor_Tantalum_SMD:CP_EIA-1608-08_AVX-J_HandSolder, symbol Device:C_Polarized
- added C28: 1.8 pF, Capacitor_SMD:C_0201_0603Metric, symbol Device:C
- added C30, C32: 4.7 uF, Capacitor_SMD:C_0201_0603Metric, symbol Device:C
- added C31: 1.5 pF, Capacitor_SMD:C_0201_0603Metric, symbol Device:C
- added C33, C36: 0.1 uF, Capacitor_SMD:C_0201_0603Metric, symbol Device:C
- added C5, C6: 6 pF, Capacitor_SMD:C_0201_0603Metric_Pad0.64x0.40mm_HandSolder, symbol Device:C
- added D1: SD03_SOD323, Diode_SMD:D_SOD-323, symbol Diode:SD05_SOD323
- added D2: BAT54C, Package_TO_SOT_SMD:SOT-23, symbol Diode:BAT54C
- added D3: D, symbol Device:D
- added D4, D5: LED, LED_SMD:LED_0805_2012Metric, symbol Device:LED
- added E1: AMCA31-2R450G-S1F-T3, AMCA31_2R450G_S1F_T3:XDCR_AMCA31-2R450G-S1F-T3, symbol AMCA31-2R450G-S1F-T3:AMCA31-2R450G-S1F-T3
- added J1: 12402012E212A, 12402012E212A:AMPHENOL_12402012E212A, symbol 12402012E212A:12402012E212A
- added J2: S2B-PH-K-SLFSN, Connector_JST:JST_ZH_B2B-ZR_1x02_P1.50mm_Vertical, symbol jst:S2B-PH-K-SLFSN
- added J3: Conn_01x03_Pin, Connector_JST:JST_ZH_B3B-ZR_1x03_P1.50mm_Vertical, symbol Connector:Conn_01x03_Pin
- added J4: Conn_01x08_Pin, symbol Connector:Conn_01x08_Pin
- added L1: 2.0 nH, Inductor_SMD:L_0201_0603Metric_Pad0.64x0.40mm_HandSolder, symbol Device:L
- added L3: 3.9 nH, Inductor_SMD:L_0201_0603Metric, symbol Device:L
- added LS2: CMT-0525-75-SMT-TR, CMT_0525_75_SMT_TR:XDCR_CMT-0525-75-SMT-TR, symbol CMT-0525-75-SMT-TR:CMT-0525-75-SMT-TR
- added Q2: NPN, Package_TO_SOT_SMD:SOT-723, symbol Simulation_SPICE:NPN
- added R1: 0, Resistor_SMD:R_0201_0603Metric_Pad0.64x0.40mm_HandSolder, symbol Device:R_US
- added R10, R15, R7, R8, R9: 10 K, Resistor_SMD:R_0201_0603Metric_Pad0.64x0.40mm_HandSolder, symbol Device:R_US
- added R11: 220, Resistor_SMD:R_0201_0603Metric_Pad0.64x0.40mm_HandSolder, symbol Device:R_US
- added R12: 470, Resistor_SMD:R_0201_0603Metric_Pad0.64x0.40mm_HandSolder, symbol Device:R_US
- added R13: 2k, Resistor_SMD:R_0201_0603Metric_Pad0.64x0.40mm_HandSolder, symbol Device:R_US
- added R19, R2, R3, R4, R5, R6: 5 K, Resistor_SMD:R_0201_0603Metric_Pad0.64x0.40mm_HandSolder, symbol Device:R_US
- added SW2, SW3: PTS810_SJM_250_SMTR_LFS, PTS810SJM250SMTR_LFS:SW_PTS810_SJM_250_SMTR_LFS, symbol PTS810_SJM_250_SMTR_LFS:PTS810_SJM_250_SMTR_LFS
- added U1: ESP32-S3, ESP32_S3:IC_ESP32-S3, symbol ESP32-S3:ESP32-S3
- added U10: LP38691SD-3.3, LP38691SD_3_3_NOPB:DFN300X300X80-7N, symbol LP38691SD-3.3:LP38691SD-3.3
- added U11: BME688, BME688:IC_BME688, symbol BME688:BME688
- added U12: RV-3028-C7_32.768KHZ_1PPM-TA-QC, Package_SON:MicroCrystal_C7_SON-8_1.5x3.2mm_P0.9mm, symbol RV-3028-C7_32.768KHZ_1PPM-TA-QC:RV-3028-C7_32.768KHZ_1PPM-TA-QC
- added U13: LTR-329ALS-01, LTR_329ALS_01:IC_LTR-329ALS-01, symbol LTR-329ALS-01:LTR-329ALS-01
- added U15: MCP73832T-2ACI/MC, MCP73832T:DFN8_2x3MC_MCH-L, symbol MCP73832T_2ACI:MCP73832T-2ACI_MC
- added U16: LSM6DSO32TR, LSM6DSO32TR:XDCR_LSM6DSO32TR, symbol LSM6DSO32TR:LSM6DSO32TR
- added U2: MX25R6435FZAIH0, MX25R6435FZAIH0:SON80P400X400X60-9N, symbol MX25R6435FZAIH0:MX25R6435FZAIH0
- added U3: DRV2605LYZFR, DRV2605LYZFR:YZF0009ADAD, symbol DRV2605LYZFR:DRV2605LYZFR
- added U4: MLX90393SLW-ABA-011-RE, MLX90393SLW_ABA_011_RE:QFN50P300X300X100-17N, symbol MLX90393SLW-ABA-011-RE:MLX90393SLW-ABA-011-RE
- added U5: MAX17048G_T10, MAX17048G_T10:SON50P200X200X80-9N, symbol MAX17048G_T10:MAX17048G_T10
- added U6: TMC6300-LA-T, tcm6300:21-100586_K2033&plus_1C_ADI-M, symbol tcm6300:TMC6300-LA-T
- added U8: USBLC6-2SC6, Package_TO_SOT_SMD:SOT-23-6, symbol Power_Protection:USBLC6-2SC6
- added Y1: ABM12W-40.0000MHZ-8-B1U-T3, ABM12W_40_0000MHZ_8_B1U_T3:XTAL_ABM12W-40.0000MHZ-8-B1U-T3, symbol ABM12W-40.0000MHZ-8-B1U-T3:ABM12W-40.0000MHZ-8-B1U-T3
- C1: value 0.1uF -> 1 uF; footprint Capacitor_SMD:C_0603_1608Metric_Pad1.08x0.95mm_HandSolder -> Capacitor_SMD:C_0201_0603Metric_Pad0.64x0.40mm_HandSolder
Connections:
- net +BATT: now also C32.2, C33.2, D2.2, J2.1, U5.2 (CELL)
- net DO: now also U4.5 (SDA/MOSI), U4.6 (MISO)
- net ENCODER: now also U4.2 (MS/CS)
- net GND: now also C10.2, C11.2, C12.2, C13.2, C14.2, C15.2, C16.2, C17.2, C18.2, C19.2, C2.2, C20.2, C21.1, C22.2, C23.2, C25.2, C26.2, C27.1, C28.1, C29.1, C3.2, C30.1, C31.1, C32.1, C33.1, C36.1, C37.2, C4.2, C5.1, C6.1, C7.2, C8.2, C9.2, D1.1 (A1), D5.1 (K), J1.A1_B12 (GND), J1.B1_A12 (GND__1), J2.2, Q2.3 (E), R10.1, R13.2, R15.2, R4.2, R5.1, SW2.2, SW3.2, U1.57 (GND), U10.2 (GND), U11.1 (GND), U11.5 (SDO), U11.7 (GND__1), U12.5 (VSS), U13.2 (GND), U15.6 (VSS), U15.9 (EP), U16.2 (SDX), U16.3 (SCX), U16.6 (GND), U16.7 (GND__1), U2.4 (GND), U3.B3 (GND), U4.1 (INT), U4.11 (A1), U4.12 (A0), U4.13 (VSS), U4.7 (INT/TRIG), U5.1 (CTG), U5.4 (GND), U5.6 (QSTRT), U5.9 (EP), U6.14 (GND), U6.16 (BRUV), U6.20 (BRW), U6.21 (GND), U6.8 (GND), U6.9 (GND), U8.2 (GND), Y1.2 (GND), Y1.4 (GND__1)
- net SCLK: now also U4.3 (SCL/SCLK)
- net U: now also J3.1 (Pin_1), U6.15 (U)
- net USR_BUTT: now also C37.1, R19.2; no longer C1.1
- net V: now also J3.2 (Pin_2), U6.17 (V)
- net W: now also J3.3 (Pin_3), U6.1 (W)
- new net: C28.2, E1.1, L3.1
- new net: R15.1, U12.6 (VBACKUP)
- new net: D5.2 (A), R11.2
- new net: J1.B5 (CC1_B), R4.1
- new net: C5.2, R1.1, Y1.1
- new net: J1.A5 (CC1_A), R5.2
- new net: Q2.2 (B), R6.1
- new net: C21.2, U3.A2 (REG)
- new net: C22.1, U6.13 (1.8VOUT)
- new net: D4.1 (K), R12.2
- new net: D3.2 (A), LS2.N, Q2.1 (C)
- new net: R12.1, U15.5 (STAT)
- new net: R13.1, U15.8 (PROG)
- new net +3.3V: C10.1, C11.1, C13.1, C14.1, C15.1, C16.1, C2.1, C20.1, C23.1, C27.2, C3.1, C36.2, C4.1, C8.1, C9.1, D1.2 (A2), D3.1 (K), L1.1, LS2.P, R19.1, R2.1, R3.1, R7.2, R8.2, R9.2, U1.20 (VDD3P3_RTC), U1.46 (VDD3P3_CPU), U1.55 (VDDA1), U1.56 (VDDA2), U10.4 (VOUT), U10.5 (SNS), U11.2 (CSB), U11.6 (VDDIO), U11.8 (VDD), U12.7 (VDD), U13.1 (VDD), U16.1 (SDO/SA0), U16.12 (CS), U16.5 (VDDIO), U16.8 (VDD), U4.15 (VDD), U4.8 (VDD_IO), U5.3 (VDD), U6.11 (VIO/NSTDBY)
- new net +3.3VA: C12.1, L1.2, U1.2 (VDD3P3), U1.3 (VDD3P3__1)
- new net +5V: C17.1, C24.1, C25.1, C26.1, C29.2, D2.3, U10.1 (VIN_2), U10.6 (VIN), U3.C2 (VDD), U6.18 (VS)
- new net +5VA: C30.2, D2.1, D4.2 (A), J1.A4_B9 (VBUS), J1.B4_A9 (VBUS__1), U15.1 (VDD), U15.2 (VDD), U8.5 (VBUS)
- new net +BAT1: U15.3 (VBAT), U15.4 (VBAT)
- new net 17: U1.23 (GPIO17)
- new net 18: U1.24 (GPIO18)
- new net 21: U1.27 (GPIO21)
- new net 33: U1.38 (GPIO33)
- new net 34: U1.39 (GPIO34)
- new net 35: U1.40 (GPIO35)
- new net 36: U1.41 (GPIO36)
- new net 37: U1.42 (GPIO37)
- new net 38: U1.43 (GPIO38)
- new net 39: U1.44 (MTCK)
- new net 40: U1.45 (MTDO)
- new net 41: U1.47 (MTDI)
- new net 42: U1.48 (MTMS)
- new net 45: U1.51 (GPIO45)
- new net 46: U1.52 (GPIO46)
- new net 47: U1.37 (SPICLK_P)
- new net 48: U1.36 (SPICLK_N)
- new net Boot: C18.1, R2.2, SW2.3, U1.5 (GPIO0)
- new net Buzzer: R6.2, U1.18 (GPIO13)
- new net CLK: U12.1 (CLKOUT)
- new net DIAG: U1.17 (GPIO12), U6.12 (DIAG)
- new net EVI: R10.2, U12.8 (EVI)
- new net Gauge: U5.5 (~{ALERT})
- new net HMN: U3.C3 (OUT-)
- new net HMP: U3.A3 (OUT+)
- new net Haptic: U1.10 (GPIO5), U3.A1 (EN)
- new net Haptic_trigg: U3.B1 (IN_TRIG)
- new net INT1: U16.4 (INT1)
- new net INT2: U16.9 (INT2)
- new net LED: R11.1, U1.6 (GPIO1)
- new net LNA_IN: C31.2, L3.2, U1.1 (LNA_IN)
- new net MFP: U1.9 (GPIO4)
- new net RGB LED: U1.19 (GPIO14)
- new net RTC: R9.1, U12.2 (~{INT})
- new net RTC_CLK: U1.21 (XTAL_32K_P)
- new net RX: U1.50 (U0RXD)
- new net Reset: C19.1, R3.2, SW3.3, U1.4 (CHIP_PU)
- new net SCL: R8.1, U1.7 (GPIO2), U11.4 (SCK), U12.3 (SCL), U13.4 (SCL), U16.13 (SCL), U3.C1 (SCL), U5.7 (SCL)
- new net SDA: R7.1, U1.8 (GPIO3), U11.3 (SDI), U12.4 (SDA), U13.3 (SDA), U16.14 (SDA), U3.B2 (SDA), U5.8 (SDA)
- new net SPI_CLK: U1.33 (SPICLK), U2.6 (SCLK)
- new net SPI_CS0: U1.32 (SPICS0), U2.1 (CS#)
- new net SPI_D: U1.35 (SPID), U2.5 (SI/SIO0)
- new net SPI_HD: U1.30 (SPIHD), U2.7 (RESET#/SIO3)
- new net SPI_Q: U1.34 (SPIQ), U2.2 (SO/SIO1)
- new net SPI_WP: U1.31 (SPIWP), U2.3 (WP#/SIO2)
- new net TX: U1.49 (U0TXD)
- new net UH: U1.16 (GPIO11), U6.3 (UH)
- new net UL: U1.13 (GPIO8), U6.6 (UL)
- new net USB_DN: U1.25 (GPIO19), U8.3 (I/O2)
- new net USB_DN1: J1.A7 (D-_A), J1.B7 (D-_B), U8.4 (I/O2)
- new net USB_DP: U1.26 (GPIO20), U8.1 (I/O1)
- new net USB_DP1: J1.A6 (D+_A), J1.B6 (D+_B), U8.6 (I/O1)
- new net VCP: C24.2, U6.2 (VCP)
- new net VDD_SPI: C1.1, C7.1, U1.29 (VDD_SPI), U2.8 (VCC)
- new net VH: U1.15 (GPIO10), U6.4 (VH)
- new net VL: U1.11 (GPIO6), U6.10 (VL)
- new net WH: U1.14 (GPIO9), U6.5 (WH)
- new net WL: U1.12 (GPIO7), U6.7 (WL)
- new net XTAL_N: C6.2, U1.53 (XTAL_N), Y1.3
- new net XTAL_P: R1.2, U1.54 (XTAL_P)
- no-connect marks 6 -> 16
Other:
- note added: "Antenna"
- note added: "Battery control"
- note added: "Buzzer"
- note added: "Crystals"
- note added: "Encoder"
- note added: "Flash and PSRAM(optional)"
- note added: "Haptic engine"
- note added: "I2C"
- note added: "IMU"
- note added: "Light sensor"
- note added: "Microcontroller"
- note added: "Motor"
- note added: "Power supply"
- note added: "RGB"
- note added: "RTC module"
- note added: "Temp and humidity"
- note added: "USB"
- note added: "User interaction"
- note added: "battery charger"
- note added: "battery gauge"
- note added: "button must be connected to pin capable of pull up"
- note added: "could add current sensing and on/off control if needed"

Commit message: start routing on bottom pcb
Parts:
- removed J4: Conn_01x08_Pin, symbol Connector:Conn_01x08_Pin
- added J4, J5: Conn_01x04_Pin, Connector_PinHeader_1.27mm:PinHeader_1x04_P1.27mm_Vertical, symbol Connector:Conn_01x04_Pin
Connections:
- net 17 is gone; now on net EVI: U1.23 (GPIO17)
- net CLK is gone; now on net RTC_CLK: U12.1 (CLKOUT)
- net +3.3V: now also J4.1 (Pin_1)
- net DO: no longer U4.5 (SDA/MOSI), U4.6 (MISO)
- net GND: now also J4.2 (Pin_2)
- net RTC: now also U1.22 (XTAL_32K_N)
- net SCLK: now also J5.2 (Pin_2)
- new net BACKLIGHT_EN: J4.3 (Pin_3)
- new net DC: J4.4 (Pin_4)
- new net MISO: U4.6 (MISO)
- new net MOSI: J5.3 (Pin_3), U4.5 (SDA/MOSI)
- new net nCS: J5.1 (Pin_1)
- new net nRESET: J5.4 (Pin_4)
Other:
- note added: "MOSI AND DO ARE THE SAME?"

Commit message: connections for bottom pcb
Parts:
- added J6: Conn_01x02_Pin, Connector_JST:JST_ZH_B2B-ZR_1x02_P1.50mm_Vertical, symbol Connector:Conn_01x02_Pin
- D3: footprint (none) -> Diode_SMD:D_0201_0603Metric_Pad0.64x0.40mm_HandSolder
Connections:
- net +BAT1 is gone; now on net +BATT: U15.3 (VBAT), U15.4 (VBAT)
- net 38 is gone; now on net Haptic_trigg: U1.43 (GPIO38)
- net 39 is gone; now on net Haptic: U1.44 (MTCK)
- net 40 is gone; now on net Gauge: U1.45 (MTDO)
- net 41 is gone; now on net MISO: U1.47 (MTDI)
- net 42 is gone; now on net MOSI: U1.48 (MTMS)
- net 45 is gone; now on net SCLK: U1.51 (GPIO45)
- net 46 is gone; now on net ENCODER: U1.52 (GPIO46)
- net MFP is gone; now on net Buzzer: U1.9 (GPIO4)
- net Boot: now also SW2.4
- net Buzzer: no longer U1.18 (GPIO13)
- net GND: now also SW2.1, SW3.1
- net HMN: now also J6.2 (Pin_2)
- net HMP: now also J6.1 (Pin_1)
- net Haptic: no longer U1.10 (GPIO5)
- net Reset: now also SW3.4
- net U: now also J3.3 (Pin_3); no longer J3.1 (Pin_1)
- net W: now also J3.1 (Pin_1); no longer J3.3 (Pin_3)

Commit message: things to improve
Other:
- note added: "Change size from 0201 to 0403 hand soldering"
- note added: "tvs should be on the input of the power supply"
Changed lines of the file:
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@@
+		)
+	)
+	(text "tvs should be on the input of the power supply\n"
+		(exclude_from_sim no)
+		(at 375.412 144.018 0)
+		(effects
+			(font
+				(size 1.27 1.27)
+			)
 		)
 	)
@@
 			)
 		)
+	)
+	(text "Change size from 0201 to 0403 hand soldering"
+		(exclude_from_sim no)
+		(at 54.102 63.754 0)
+		(effects
+			(font
+				(size 1.27 1.27)
+			)
+		)

Commit message: I think its ready again
Parts:
- removed D1: SD03_SOD323, Diode_SMD:D_SOD-323, symbol Diode:SD05_SOD323
- C1, C10, C11, C12, C13, C14, C15, C17, C18, C19, C20, C22, C23, C24, C25, C27, C3, C37, C4, C5, C6, C7, C8, C9: footprint Capacitor_SMD:C_0201_0603Metric_Pad0.64x0.40mm_HandSolder -> Capacitor_SMD:C_0402_1005Metric_Pad0.74x0.62mm_HandSolder
- C21, C29, C30, C32, C33, C36: footprint Capacitor_SMD:C_0201_0603Metric -> Capacitor_SMD:C_0402_1005Metric_Pad0.74x0.62mm_HandSolder
- C28: footprint Capacitor_SMD:C_0201_0603Metric -> Capacitor_SMD:C_0201_0603Metric_Pad0.64x0.40mm_HandSolder; now fitted
- C31: footprint Capacitor_SMD:C_0201_0603Metric -> Capacitor_SMD:C_0201_0603Metric_Pad0.64x0.40mm_HandSolder
- D3: footprint Diode_SMD:D_0201_0603Metric_Pad0.64x0.40mm_HandSolder -> Diode_SMD:D_0402_1005Metric_Pad0.77x0.64mm_HandSolder
- L1: footprint Inductor_SMD:L_0201_0603Metric_Pad0.64x0.40mm_HandSolder -> Inductor_SMD:L_0402_1005Metric_Pad0.77x0.64mm_HandSolder
- L3: footprint Inductor_SMD:L_0201_0603Metric -> Inductor_SMD:L_0201_0603Metric_Pad0.64x0.40mm_HandSolder
- R1, R10, R11, R12, R13, R15, R19, R2, R3, R4, R5, R6, R7, R8, R9: footprint Resistor_SMD:R_0201_0603Metric_Pad0.64x0.40mm_HandSolder -> Resistor_SMD:R_0402_1005Metric_Pad0.72x0.64mm_HandSolder
Connections:
- net 34 is gone; now on net DC: U1.39 (GPIO34)
- net 35 is gone; now on net BACKLIGHT_EN: U1.40 (GPIO35)
- net 36 is gone; now on net nCS: U1.41 (GPIO36)
- net 37 is gone; now on net nRESET: U1.42 (GPIO37)
- net 47 is gone; now on net INT1: U1.37 (SPICLK_P)
- net 48 is gone; now on net INT2: U1.36 (SPICLK_N)
- net 21: no longer names the net of U1.27 (GPIO21)
- net 33: no longer names the net of U1.38 (GPIO33)
- no-connect marks 16 -> 20
Other:
- note removed: "Change size from 0201 to 0403 hand soldering"
- note removed: "MOSI AND DO ARE THE SAME?"
- note removed: "RGB"
- note removed: "button must be connected to pin capable of pull up"
- note removed: "tvs should be on the input of the power supply"
- moved on the sheet: C16

Commit message: starting to add MPN
Parts:
- E1: MPN (none) -> AMCA31-2R450G-S1F-T3
- J1: MPN (none) -> 12402012E212A
- LS2: MPN (none) -> CMT-0525-75-SMT-TR
- U1: MPN (none) -> ESP32-S3
- U10: MPN LP38691SD-3.3 -> LP38691SD-3.3/NOPB
- U11: MPN (none) -> BME688
- U12: MPN (none) -> RV-3028-C7 32.768KHZ 1PPM-TA-QC
- U13: MPN (none) -> LTR-329ALS-01
- U15: MPN (none) -> MCP73832T-2ACI/MC
- U16: MPN (none) -> LSM6DSO32TR
- U2: MPN (none) -> MX25R6435FZAIH0
- U3: MPN (none) -> DRV2605LYZFR
- U4: MPN (none) -> MLX90393SLW-ABA-011-RE
- U5: MPN (none) -> MAX17048G+T10
- U6: MPN 175-TMC6300-LA-TCT-ND -> TMC6300-LA-T
- U8: Link (none) -> https://www.digikey.es/es/products/detail/stmicroelectronic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; MPN (none) -> USBLC6-2SC6
- Y1: MPN (none) -> ABM12W-40.0000MHZ-8-B1U-T3
Changed lines of the file:
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@@
 			)
 		)
+		(property "MPN" "MAX17048G+T10"
+			(at 120.65 208.28 0)
+			(effects
+				(font
+					(size 1.27 1.27)
+				)
+				(hide yes)
+			)
+		)
 		(pin "2"
 		)
@@
 			)
 		)
+		(property "MPN" "AMCA31-2R450G-S1F-T3"
+			(at 212.09 229.87 0)
+			(effects
+				(font
+					(size 1.27 1.27)
+				)
+				(hide yes)
+			)
+		)
 		(pin "1"
 		)
@@
 			)
 		)
+		(property "MPN" "ABM12W-40.0000MHZ-8-B1U-T3"
+			(at 549.91 64.77 0)
+			(effects
+				(font
+					(size 1.27 1.27)
+				)
+				(hide yes)
+			)
+		)
 		(pin "1"
 		)
@@
 			)
 		)
-		(property "MPN" "LP38691SD-3.3"
+		(property "MPN" "LP38691SD-3.3/NOPB"
 			(at 368.3 162.56 0)
 			(effects
@@
 			)
 		)
+		(property "MPN" "LSM6DSO32TR"
+			(at 105.41 124.46 0)
+			(effects
+				(font
+					(size 1.27 1.27)
+				)
+				(hide yes)
+			)
+		)
 		(pin "1"
 		)
@@
 			)
 		)
+		(property "MPN" "  BME688"
+			(at 118.11 50.8 0)
+			(effects
+				(font
+					(size 1.27 1.27)
+				)
+				(hide yes)
+			)
+		)
 		(pin "8"
 		)
@@
 			)
 		)
+		(property "MPN" "ESP32-S3"
+			(at 505.46 283.21 0)
+			(effects
+				(font
+					(size 1.27 1.27)
+				)
+				(hide yes)
+			)
+		)
 		(pin "2"
 		)
@@
 			)
 		)
+		(property "MPN" "12402012E212A"
+			(at 353.06 234.95 0)
+			(effects
+				(font
+					(size 1.27 1.27)
+				)
+				(hide yes)
+			)
+		)
 		(pin "B4_A9"
 		)
@@
 			)
 		)
+		(property "MPN" "DRV2605LYZFR"
+			(at 228.6 309.88 0)
+			(effects
+				(font
+					(size 1.27 1.27)
+				)
+				(hide yes)
+			)
+		)
 		(pin "A2"
 		)
@@
 			)
 		)
-		(property "MPN" "175-TMC6300-LA-TCT-ND"
+		(property "MPN" "  TMC6300-LA-T"
 			(at 191.77 46.99 0)
 			(effects
@@
 			)
 		)
+		(property "MPN" "USBLC6-2SC6"
+			(at 417.83 224.79 0)
+			(effects
+				(font
+					(size 1.27 1.27)
+				)
+				(hide yes)
+			)
+		)
+		(property "Link" "https://www.digikey.es/es/products/detail/stmicroelectronics/USBLC6-2SC6/1040559"
+			(at 417.83 224.79 0)
+			(effects
+				(font
+					(size 1.27 1.27)
+				)
+				(hide yes)
+			)
+		)
 		(pin "5"
 		)
@@
 			)
 		)
+		(property "MPN" "CMT-0525-75-SMT-TR"
+			(at 386.08 313.69 0)
+			(effects
+				(font
+					(size 1.27 1.27)
+				)
+				(hide yes)
+			)
+		)
 		(pin "N"
 		)
@@
 			)
 		)
+		(property "MPN" "RV-3028-C7 32.768KHZ 1PPM-TA-QC"
+			(at 217.17 166.37 0)
+			(effects
+				(font
+					(size 1.27 1.27)
+				)
+				(hide yes)
+			)
+		)
 		(pin "1"
 		)
@@
 			)
 		)
+		(property "MPN" "MCP73832T-2ACI/MC"
+			(at 29.21 196.85 0)
+			(effects
+				(font
+					(size 1.27 1.27)
+				)
+				(hide yes)
+			)
+		)
 		(pin "4"
 		)
@@
 			)
 		)
+		(property "MPN" "LTR-329ALS-01"
+			(at 335.28 73.66 90)
+			(effects
+				(font
+					(size 1.27 1.27)
+				)
+				(hide yes)
+			)
+		)
 		(pin "1"
 		)
@@
 			)
 		)
+		(property "MPN" "MX25R6435FZAIH0"
+			(at 495.3 170.18 0)
+			(effects
+				(font
+					(size 1.27 1.27)
+				)
+				(hide yes)
+			)
+		)
 		(pin "7"
 		)
@@
 				(hide yes)
 			)
+		)
+		(property "MPN" "MLX90393SLW-ABA-011-RE"
+			(at 78.74 303.53 0)
+			(effects
+				(font
+					(size 1.27 1.27)
+				)
+				(hide yes)
+			)
